File: Hardware/titan_2022/titan_2022.kicad_sch (KiCad schematic)
At the start: 73 parts, among them J1 SEC_{OUT}, J10 Conn_02x20_Odd_Even, J2 SEC_{IN}, J3 SWD, J4 BATTERY, J5 MONITOR, J6 DHT, J7 CO_{2}, J8 WHEELS, J9 USB_B_Mini, Q1 DMG2301L, SW1 RPON, SW2 SHTDN, SW3 MCU_RST, U1 NRF24L01, U2 AP62301WU, U3 ULT-GPS, U4 STM32F103C8Tx, Y1 8MHz

Commit message: Cleaned up schematics
Other:
- note added: "5V 3A Regulator provides 5V to the RPi. Resistor voltage division on EN pin to achieve under voltage lock out (UVLO) to protect batteries."
- note added: "Both wheels have an MLX90614 sensor to monitor brake disk temeprature, the rear has an IR reflectometer used as an optical encoder for distance and speed. These sensors provide data over I2C and a digital line respectively."
- note added: "Collects and distributes bike data between RPi systems using UART to communicate with RPis. Can be programmed and debugged either by UART through the RPi or USB. SWD header also added for programming without USB support. RPi it is mounted to connects by UART1, the other on UART3. There is a button to reset specifically the MCU. There are a few controlled status LEDs."
- note added: "Connections for secondary board to connect to main board."
- note added: "Digital CO_{2} sensor that measures up to 2000ppm using infrared. Outputs level using PWM. Sensor is placed near the riders' heads."
- note added: "Digital temperature and humidity sensor used to derive ambient air conditions for performance calculations. Sensor is placed near the air intake."
- note added: "GPS is used primarily as a backup source for distance and speed information but location can also be recorded during the run."
- note added: "MH-Z19 (CO_{2})"
- note added: "Mainly used for providing power to the RPi, drawing 3.3V from the RPi for the HAT, and exchanging data over UART."
- note added: "Power from LiFePO_{4} batteries is fed through a reverse polarity protectioncircuit, then to the monitor power pads and the 5V regulator."
- note added: "Pullups for long I2C lines"
- note added: "RPi Header"
- note added: "Sec. Input"
- note added: "Status 1 is PWM-able"
- note added: "Wheels"
- note removed: "5V 3A Regulator provides 5V to the RPi. Has a switch to ground its EN pin to restart system."
- note removed: "Collects and distributes bike data between RPi systems using UART to communicate with RPis. Can be programmed and debugged either by UART through the RPi or USB. RPi it is mounted to connects by UART1, the other on UART2. There is a button to reset specifically the MCU."
- note removed: "Connections for the main board to the secondary board and encoder."
- note removed: "Digital temperature and humidity sensor"
- note removed: "GPS is used primarily as a backup source for speed information but coordinates are recorded during the run. Connected on UART3."
- note removed: "Main Input"
- note removed: "Power is fed through a reverse polarity protection circuit, then to the monitor power pads and the 5V regulator."
- note removed: "Pullups for long I2C line"
- note removed: "Status 1 is PWMable"
- moved on the sheet: C1, C2, C3, C4, C5, D10, D11, D12, D3, D4, D5, D6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
