File: Hardware/titan_wheel/titan_wheel.kicad_pcb (KiCad board)
At the start: 2 copper layers, 48 x 20 mm, 19 parts, among them J1 REAR, J2 RPI, U1 LM358, U2 TCRT5000, U3 MLX90614

Commit message: Cleaned up schematics
Parts:
- J1: value REAR -> OTHER
- turned R2 to -90 degrees
Connections:
- R2 pad 1: +5V -> Net-(U2-PadA)
- R2 pad 2: Net-(R2-Pad2) -> +5V
- U2 pad A: Net-(R2-Pad2) -> Net-(U2-PadA)
Routing:
- net Net-(U2-PadA): track 0.00 -> 9.81 mm
- net Net-(R2-Pad2): track 9.81 -> 0.00 mm
Changed lines of the file:
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@@
   (net 5 "/SCL")
   (net 6 "+5V")
-  (net 7 "Net-(R2-Pad2)")
+  (net 7 "Net-(U2-PadA)")
   (net 8 "/REFLECTIVITY")
   (net 9 "/THRESHOLD")
@@
   )
   (footprint "Resistor_SMD:R_0603_1608Metric" (layer "F.Cu")
-    (at 165.75 51.5 90)
+    (at 165.75 51.5 -90)
     (descr "Resistor SMD 0603 (1608 Metric), square (rectangular) end terminal, IPC_7351 nominal, (Body size source: IPC-SM-782 page 72, https://www.pcb-3d.com/wordpress/wp-content/uploads/ipc-sm-782a_amendment_1_and_2.pdf), generated with kicad-footprint-generator")
     (tags "resistor")
@@
     (property "Sheetname" "")
     (attr smd)
-    (fp_text reference "R2" (at -2.5 0 90) (layer "F.SilkS")
+    (fp_text reference "R2" (at 2.5 0 90) (layer "F.SilkS")
       (effects (font (size 1 1) (thickness 0.15)))
     )
@@
     (fp_line (start 0.8 0.4125) (end -0.8 0.4125) (layer "F.Fab") (width 0.1))
     (fp_line (start 0.8 -0.4125) (end 0.8 0.4125) (layer "F.Fab") (width 0.1))
-    (pad "1" smd roundrect (at -0.825 0 90) (size 0.8 0.95) (layers "F.Cu" "F.Paste" "F.Mask") (roundrect_rratio 0.25)
+    (pad "1" smd roundrect (at -0.825 0 270) (size 0.8 0.95) (layers "F.Cu" "F.Paste" "F.Mask") (roundrect_rratio 0.25)
+      (net 7 "Net-(U2-PadA)") (pintype "passive"))
+    (pad "2" smd roundrect (at 0.825 0 270) (size 0.8 0.95) (layers "F.Cu" "F.Paste" "F.Mask") (roundrect_rratio 0.25)
       (net 6 "+5V") (pintype "passive"))
-    (pad "2" smd roundrect (at 0.825 0 90) (size 0.8 0.95) (layers "F.Cu" "F.Paste" "F.Mask") (roundrect_rratio 0.25)
-      (net 7 "Net-(R2-Pad2)") (pintype "passive"))
     (model "${KICAD6_3DMODEL_DIR}/Resistor_SMD.3dshapes/R_0603_1608Metric.wrl"
       (offset (xyz 0 0 0))
@@
       (effects (font (size 1 1) (thickness 0.15)))
     )
-    (fp_text value "REAR" (at 0 9.95 90) (layer "F.Fab")
+    (fp_text value "OTHER" (at 0 9.95 90) (layer "F.Fab")
       (effects (font (size 1 1) (thickness 0.15)))
     )
@@
     (pad "" np_thru_hole circle (at 0 -1.9 90) (size 2.5 2.5) (drill 2.5) (layers *.Cu *.Mask))
     (pad "A" thru_hole circle (at 2.75 1.27 90) (size 1.5 1.5) (drill 1) (layers *.Cu *.Mask)
-      (net 7 "Net-(R2-Pad2)") (pintype "passive"))
+      (net 7 "Net-(U2-PadA)") (pintype "passive"))
     (pad "CATH" thru_hole circle (at 2.75 -1.27 90) (size 1.5 1.5) (drill 1) (layers *.Cu *.Mask)
       (net 1 "GND") (pintype "passive"))
